Commit message: forward kinematics done

File: src/yr_description/urdf/exo.xacro (robot description, xacro)
@@ -1,15 +1,19 @@
 <?xml version="1.0"?>
-<robot name="lower_limb_exoskeleton" xmlns:xacro="http://www.ros.org/wiki/xacro">
+<robot name="exo"
+  xmlns:xacro="http://www.ros.org/wiki/xacro">
+  <xacro:property name="debug" default="false"/>
   <xacro:include filename="properties.xacro" />
   <xacro:include filename="macros.xacro" />
-  <xacro:include filename="transmissions.xacro" />\
+  <xacro:include filename="transmissions.xacro" />
+\
   <xacro:include filename="depth_cameras_setup.xacro" />
-  <link name="world"/>
-  <joint name="pole_to_waist" type="fixed">
-    <parent link="world" />
-    <child link="waist_link" />
-    <origin xyz="0 0 1.5" />
-  </joint>
-  <!-- <link name="human_waist_link">
+  <!-- <link name="world"/>
+    <joint name="pole_to_waist" type="fixed">
+        <parent link="world" />
+        <child link="waist_link" />
+        <origin xyz="0 0 1.5" />
+    </joint> -->
+  <!--
+  <link name="human_waist_link">
     <visual>
       <origin xyz="0 0 ${-human_waist_h/2}" rpy="0 0 0" />
@@ -28,11 +32,5 @@
       <origin xyz="0 0 ${-human_waist_h/2}" rpy="0 0 0" />
       <mass value="${human_waist_weight}" />
-      <inertia
-        ixx="${human_waist_weight / 12.0 * (human_waist_w**2 + human_waist_h**2)}"
-        iyy="${human_waist_weight / 12.0 * (human_waist_l**2 + human_waist_h**2)}"
-        izz="${human_waist_weight / 12.0 * (human_waist_l**2 + human_waist_w**2)}"
-        ixy="0"
-        ixz="0"
-        iyz="0" />
+      <inertia ixx="${human_waist_weight / 12.0 * (human_waist_w**2 + human_waist_h**2)}" iyy="${human_waist_weight / 12.0 * (human_waist_l**2 + human_waist_h**2)}" izz="${human_waist_weight / 12.0 * (human_waist_l**2 + human_waist_w**2)}" ixy="0" ixz="0" iyz="0" />
     </inertial>
   </link>
@@ -40,92 +38,56 @@
     <parent link="waist_link" />
     <child link="human_waist_link" />
-    <origin xyz="${human_waist_l/2 + 0.08} 0 ${human_waist_h/3}" rpy="0 0 0" />
+    <origin xyz="${human_waist_l/2 + 0.08} 0 ${0}" rpy="0 0 0" />
   </joint> -->
-  <xacro:create_link3 name="waist_link" m="${waist_m}" l="${waist_l}" w="${waist_w/2}"
-    h="${waist_h}" o_x="0" o_y="${waist_mesh_w/2 -0.015}" o_z="${-waist_h_offset}" o_r="0"
-    o_p="${-PI}"
-    o_yaw="${-PI}" mat="${waist_mat}" mesh_filename="${waist_mesh}" mirror="1" />
-  <xacro:create_link3 name="l_pel_link" m="${pel_m}" l="${pel_l}" w="${pel_w}"
-    h="${pel_h}" o_x="${pel_x_offset}" o_y="${pel_y_offset}"
-    o_z="${-pel_h_offset}" o_r="0" o_p="0"
-    o_yaw="0" mat="${pel_mat}" mesh_filename="${pel_mesh}" mirror="1" />
-  <xacro:create_link3 name="l_thigh_link" m="${thigh_m}" l="${thigh_l}" w="${thigh_w}"
-    h="${thigh_h}" o_x="${thigh_w}" o_y="${thigh_w/2}" o_z="${-thigh_l}" o_r="0" o_p="0"
-    o_yaw="${PI}" mat="${thigh_mat}" mesh_filename="${thigh_mesh}" mirror="1" />
-  <xacro:create_link3 name="l_shank_link" m="${shank_m}" l="${shank_l}" w="${shank_w}"
-    h="${shank_h}" o_x="${shank_w}" o_y="${shank_w/2}" o_z="${-shank_l}" o_r="0" o_p="0"
-    o_yaw="${PI}"
-    mat="${shank_mat}" mesh_filename="${shank_mesh}" mirror="1" />
-  <!-- <xacro:create_link2 name="l_foot_link" m="${foot_m}" l="${foot_h}" w="${foot_w}"
-    h="${foot_l}" o_x="${-foot_h}" o_y="${foot_w}" o_z="${-foot_l}" o_r="0" o_p="0" o_yaw="0"
-    mat="${foot_mat}"
-    mesh_filename="${foot_mesh}" mirror="-1" /> -->
-    <link name="l_foot_link">
-      <collision>
-        <origin xyz="${foot_h/2} 0 ${-foot_h}" rpy="0 0 0" />
-        <geometry>
-            <box size="${foot_h*2} ${foot_w} ${foot_l/2}" />
-        </geometry>
-      </collision>
-      <visual>
-              <origin xyz="${-foot_h} ${foot_w} ${-foot_l}" rpy="${PI/2} 0 ${PI/2 + 0}" />
-          <geometry>
-          <mesh filename="${foot_mesh}"
-                      scale="${-1*mesh_scale} ${mesh_scale} ${mesh_scale}" />
-          </geometry>
-          <origin xyz="0 0 ${-foot_h/2}" rpy="0 0 0" />
-          <material name="${foot_mat}" />
-      </visual>
-      <inertial>
-          <origin xyz="0 0 ${-foot_h/2}" rpy="0 0 0" />
-          <mass value="${foot_m}" />
-          <inertia
-              ixx="${foot_m / 12.0 * (foot_w*foot_w + foot_h*foot_h)}"
-              ixy="0.0" ixz="0.0"
-              iyy="${foot_m / 12.0 * (foot_l*foot_l + foot_h*foot_h)}"
-              iyz="0.0"
-              izz="${foot_m / 12.0 * (foot_l*foot_l + foot_w*foot_w)}" />
-      </inertial>
+  <xacro:create_link3 name="waist_link" m="${waist_m}" l="${waist_l}" w="${waist_w/2}" h="${waist_h}" o_x="0" o_y="${waist_mesh_w/2 -0.015}" o_z="${-waist_h_offset}" o_r="0" o_p="${-PI}" o_yaw="${-PI}" mat="${waist_mat}" mesh_filename="${waist_mesh}" mirror="1" />
+  <xacro:create_link3 name="l_pel_link" m="${pel_m}" l="${pel_l}" w="${pel_w}" h="${pel_h}" o_x="${pel_x_offset}" o_y="${pel_y_offset}" o_z="${-pel_h_offset}" o_r="0" o_p="0" o_yaw="0" mat="${pel_mat}" mesh_filename="${pel_mesh}" mirror="1" />
+  <xacro:create_link3 name="l_thigh_link" m="${thigh_m}" l="${thigh_l}" w="${thigh_w}" h="${thigh_h}" o_x="${thigh_w}" o_y="${thigh_w/2}" o_z="${-thigh_l}" o_r="0" o_p="0" o_yaw="${PI}" mat="${thigh_mat}" mesh_filename="${thigh_mesh}" mirror="1" />
+  <xacro:create_link3 name="l_shank_link" m="${shank_m}" l="${shank_l}" w="${shank_w}" h="${shank_h}" o_x="${shank_w}" o_y="${shank_w/2}" o_z="${-shank_l}" o_r="0" o_p="0" o_yaw="${PI}" mat="${shank_mat}" mesh_filename="${shank_mesh}" mirror="1" />
+  <!-- <xacro:create_link2 name="l_foot_link" m="${foot_m}" l="${foot_h}" w="${foot_w}" h="${foot_l}" o_x="${-foot_h}" o_y="${foot_w}" o_z="${-foot_l}" o_r="0" o_p="0" o_yaw="0" mat="${foot_mat}" mesh_filename="${foot_mesh}" mirror="-1" /> -->
+  <link name="l_foot_link">
+    <collision>
+      <origin xyz="${foot_h/2} 0 ${-foot_h}" rpy="0 0 0" />
+      <geometry>
+        <box size="${foot_h*2} ${foot_w} ${foot_l/2}" />
+      </geometry>
+    </collision>
+    <visual>
+      <origin xyz="${-foot_h} ${foot_w} ${-foot_l}" rpy="${PI/2} 0 ${PI/2 + 0}" />
+      <geometry>
+        <mesh filename="${foot_mesh}" scale="${-1*mesh_scale} ${mesh_scale} ${mesh_scale}" />
+      </geometry>
+      <origin xyz="0 0 ${-foot_h/2}" rpy="0 0 0" />
+      <material name="${foot_mat}" />
+    </visual>
+    <inertial>
+      <origin xyz="0 0 ${-foot_h/2}" rpy="0 0 0" />
+      <mass value="${foot_m}" />
+      <inertia ixx="${foot_m / 12.0 * (foot_w*foot_w + foot_h*foot_h)}" ixy="0.0" ixz="0.0" iyy="${foot_m / 12.0 * (foot_l*foot_l + foot_h*foot_h)}" iyz="0.0" izz="${foot_m / 12.0 * (foot_l*foot_l + foot_w*foot_w)}" />
+    </inertial>
   </link>
-  <xacro:create_link3 name="r_pel_link" m="${pel_m}" l="${pel_l}" w="${pel_w}"
-    h="${pel_h}" o_x="${pel_x_offset}" o_y="${pel_y_offset}"
-    o_z="${-pel_h_offset}" o_r="0" o_p="0"
-    o_yaw="0" mat="${pel_mat}" mesh_filename="${pel_mesh}" mirror="1" />
-  <xacro:create_link3 name="r_thigh_link" m="${thigh_m}" l="${thigh_l}" w="${thigh_w}"
-    h="${thigh_h}" o_x="${-thigh_w}" o_y="${-thigh_w/2}" o_z="${-thigh_l}" o_r="0" o_p="0"
-    o_yaw="0" mat="${thigh_mat}" mesh_filename="${thigh_mesh}" mirror="1" />
-  <xacro:create_link3 name="r_shank_link" m="${shank_m}" l="${shank_l}" w="${shank_w}"
-    h="${shank_h}" o_x="${-shank_w}" o_y="${-shank_w/2}" o_z="${-shank_l}" o_r="0" o_p="0" o_yaw="0"
-    mat="${shank_mat}" mesh_filename="${shank_mesh}" mirror="1" />
-    <!-- <xacro:create_link2 name="r_foot_link" m="${foot_m}" l="${foot_h}" w="${foot_w}"
-    h="${foot_l}" o_x="${-foot_h}" o_y="${-foot_w}" o_z="${-foot_l}" o_r="0" o_p="0" o_yaw="0"
-    mat="${foot_mat}"
-    mesh_filename="${foot_mesh}" mirror="1" /> -->
-    <link name="r_foot_link">
-      <collision>
-          <origin xyz="${foot_h/2} 0 ${-foot_h}" rpy="0 0 0" />
-          <geometry>
-              <box size="${foot_h*2} ${foot_w} ${foot_l/2}" />
-          </geometry>
-      </collision>
-      <visual>
-              <origin xyz="${-foot_h} ${-foot_w} ${-foot_l}" rpy="${PI/2} 0 ${PI/2 + 0}" />
-          <geometry>
-          <mesh filename="${foot_mesh}"
-                      scale="${1*mesh_scale} ${mesh_scale} ${mesh_scale}" />
-          </geometry>
-          <origin xyz="0 0 ${-foot_h/2}" rpy="0 0 0" />
-          <material name="${foot_mat}" />
-      </visual>
-      <inertial>
-          <origin xyz="0 0 ${-foot_h/2}" rpy="0 0 0" />
-          <mass value="${foot_m}" />
-          <inertia
-              ixx="${foot_m / 12.0 * (foot_w*foot_w + foot_h*foot_h)}"
-              ixy="0.0" ixz="0.0"
-              iyy="${foot_m / 12.0 * (foot_l*foot_l + foot_h*foot_h)}"
-              iyz="0.0"
-              izz="${foot_m / 12.0 * (foot_l*foot_l + foot_w*foot_w)}" />
-      </inertial>
+  <xacro:create_link3 name="r_pel_link" m="${pel_m}" l="${pel_l}" w="${pel_w}" h="${pel_h}" o_x="${pel_x_offset}" o_y="${pel_y_offset}" o_z="${-pel_h_offset}" o_r="0" o_p="0" o_yaw="0" mat="${pel_mat}" mesh_filename="${pel_mesh}" mirror="1" />
+  <xacro:create_link3 name="r_thigh_link" m="${thigh_m}" l="${thigh_l}" w="${thigh_w}" h="${thigh_h}" o_x="${-thigh_w}" o_y="${-thigh_w/2}" o_z="${-thigh_l}" o_r="0" o_p="0" o_yaw="0" mat="${thigh_mat}" mesh_filename="${thigh_mesh}" mirror="1" />
+  <xacro:create_link3 name="r_shank_link" m="${shank_m}" l="${shank_l}" w="${shank_w}" h="${shank_h}" o_x="${-shank_w}" o_y="${-shank_w/2}" o_z="${-shank_l}" o_r="0" o_p="0" o_yaw="0" mat="${shank_mat}" mesh_filename="${shank_mesh}" mirror="1" />
+  <!-- <xacro:create_link2 name="r_foot_link" m="${foot_m}" l="${foot_h}" w="${foot_w}" h="${foot_l}" o_x="${-foot_h}" o_y="${-foot_w}" o_z="${-foot_l}" o_r="0" o_p="0" o_yaw="0" mat="${foot_mat}" mesh_filename="${foot_mesh}" mirror="1" /> -->
+  <link name="r_foot_link">
+    <collision>
+      <origin xyz="${foot_h/2} 0 ${-foot_h}" rpy="0 0 0" />
+      <geometry>
+        <box size="${foot_h*2} ${foot_w} ${foot_l/2}" />
+      </geometry>
+    </collision>
+    <visual>
+      <origin xyz="${-foot_h} ${-foot_w} ${-foot_l}" rpy="${PI/2} 0 ${PI/2 + 0}" />
+      <geometry>
+        <mesh filename="${foot_mesh}" scale="${1*mesh_scale} ${mesh_scale} ${mesh_scale}" />
+      </geometry>
+      <origin xyz="0 0 ${-foot_h/2}" rpy="0 0 0" />
+      <material name="${foot_mat}" />
+    </visual>
+    <inertial>
+      <origin xyz="0 0 ${-foot_h/2}" rpy="0 0 0" />
+      <mass value="${foot_m}" />
+      <inertia ixx="${foot_m / 12.0 * (foot_w*foot_w + foot_h*foot_h)}" ixy="0.0" ixz="0.0" iyy="${foot_m / 12.0 * (foot_l*foot_l + foot_h*foot_h)}" iyz="0.0" izz="${foot_m / 12.0 * (foot_l*foot_l + foot_w*foot_w)}" />
+    </inertial>
   </link>
   <!-- ======================================================= -->
@@ -134,52 +96,34 @@
   <xacro:macro name="create_leg" params="side origin_y o_roll hip_y_offset">
     <xacro:if value="${side == 'l'}">
-      <xacro:property name="pel_lower_limit" value="${-PI}" />
-      <xacro:property name="pel_upper_limit" value="${-PI/4}" />
+      <xacro:property name="pel_lower_limit" value="${-PI/2}" />
+      <xacro:property name="pel_upper_limit" value="${PI/2}" />
+      <xacro:property name="pel_offset" value="${-PI/2}" />
     </xacro:if>
     <xacro:if value="${side == 'r'}">
-      <xacro:property name="pel_lower_limit" value="${PI/4}" />
-      <xacro:property name="pel_upper_limit" value="${PI}" />
+      <xacro:property name="pel_lower_limit" value="${-PI/2}" />
+      <xacro:property name="pel_upper_limit" value="${PI/2}" />
+      <xacro:property name="pel_offset" value="${PI/2}" />
     </xacro:if>
-    <xacro:create_joint2 name="yr_${side}_pel_joint" parent="waist_link"
-      child="${side}_pel_link" origin_x="0" origin_y="${origin_y}"
-      origin_z="0" o_roll="0"
-      o_pitch="0" o_yaw="${-PI}"
-      axis_x="1" axis_y="0" axis_z="0"
-      lower_limit="${pel_lower_limit}" upper_limit="${pel_upper_limit}" effort="1000" velocity="10.0" />
-    <xacro:create_joint2 name="yr_${side}_hip_joint" parent="${side}_pel_link"
-      child="${side}_thigh_link"
-      origin_x="${-pel_l}" origin_y="${hip_y_offset}" origin_z="${-pel_h}" o_roll="${o_roll}"
-      o_pitch="0" o_yaw="${-PI}"
-      axis_x="0" axis_y="1" axis_z="0"
-      lower_limit="${3*PI/4}" upper_limit="${-3*PI/4}" effort="1000" velocity="10.0" />
-    <xacro:create_joint2 name="yr_${side}_kne_joint" parent="${side}_thigh_link"
-      child="${side}_shank_link"
-      origin_x="0" origin_y="0" origin_z="${-thigh_l}" o_roll="0" o_pitch="0" o_yaw="0"
-      axis_x="0" axis_y="1" axis_z="0"
-      lower_limit="${-PI/4}" upper_limit="${3*PI/2}" effort="1000" velocity="10.0" />
-    <xacro:create_joint2 name="yr_${side}_ank_joint" parent="${side}_shank_link"
-      child="${side}_foot_link"
-      origin_x="0" origin_y="0" origin_z="${-shank_l}" o_roll="0" o_pitch="0" o_yaw="0"
-      axis_x="0" axis_y="1" axis_z="0"
-      lower_limit="${-PI}" upper_limit="${PI}" effort="1000" velocity="10.0" />
+    <xacro:create_joint name="yr_${side}_pel_joint" parent="waist_link" child="${side}_pel_link" origin_x="0" origin_y="${origin_y}" origin_z="0" o_roll="${pel_offset}" o_pitch="0" o_yaw="${-PI}" axis_x="1" axis_y="0" axis_z="0" lower_limit="${pel_lower_limit}" upper_limit="${pel_upper_limit}" effort="1000" velocity="10.0" />
+    <xacro:create_joint name="yr_${side}_hip_joint" parent="${side}_pel_link" child="${side}_thigh_link" origin_x="${-pel_l}" origin_y="${hip_y_offset}" origin_z="${-pel_h}" o_roll="${o_roll}" o_pitch="0" o_yaw="${-PI}" axis_x="0" axis_y="1" axis_z="0" lower_limit="${-3*PI/4}" upper_limit="${3*PI/4}" effort="1000" velocity="10.0" />
+    <xacro:create_joint name="yr_${side}_kne_joint" parent="${side}_thigh_link" child="${side}_shank_link" origin_x="0" origin_y="0" origin_z="${-thigh_l}" o_roll="0" o_pitch="0" o_yaw="0" axis_x="0" axis_y="1" axis_z="0" lower_limit="${-PI/4}" upper_limit="${PI}" effort="1000" velocity="10.0" />
+    <xacro:create_joint name="yr_${side}_ank_joint" parent="${side}_shank_link" child="${side}_foot_link" origin_x="0" origin_y="0" origin_z="${-shank_l}" o_roll="0" o_pitch="0" o_yaw="0" axis_x="0" axis_y="1" axis_z="0" lower_limit="${-PI/4}" upper_limit="${PI/2}" effort="1000" velocity="10.0" />
   </xacro:macro>
-  <xacro:create_leg side="l" origin_y="${(abduction_motor_distance) / 2}" o_roll="${-PI/2}"
-    hip_y_offset="${-pel_w/2}" />
-  <xacro:create_leg side="r" origin_y="${-(abduction_motor_distance) / 2}" o_roll="${PI/2}"
-    hip_y_offset="${pel_w/2}" />
- <gazebo>
-  <plugin name="gazebo_ros_control" filename="libgazebo_ros_control.so">
-    <robotNamespace>/exo</robotNamespace>
-    <robotSimType>gazebo_ros_control/DefaultRobotHWSim</robotSimType>
-  </plugin>
-</gazebo>
- <xacro:insert_transmission name="yr_l_pel_joint"/>
- <xacro:insert_transmission name="yr_l_hip_joint"/>
- <xacro:insert_transmission name="yr_l_kne_joint"/>
- <xacro:insert_transmission name="yr_l_ank_joint"/>
- <xacro:insert_transmission name="yr_r_pel_joint"/>
- <xacro:insert_transmission name="yr_r_hip_joint"/>
- <xacro:insert_transmission name="yr_r_kne_joint"/>
- <xacro:insert_transmission name="yr_r_ank_joint"/>
+  <xacro:create_leg side="l" origin_y="${(abduction_motor_distance) / 2}" o_roll="${-PI/2}" hip_y_offset="${-pel_w/2}" />
+  <xacro:create_leg side="r" origin_y="${-(abduction_motor_distance) / 2}" o_roll="${PI/2}" hip_y_offset="${pel_w/2}" />
+  <gazebo>
+    <plugin name="gazebo_ros_control" filename="libgazebo_ros_control.so">
+      <robotNamespace>/exo</robotNamespace>
+      <robotSimType>gazebo_ros_control/DefaultRobotHWSim</robotSimType>
+    </plugin>
+  </gazebo>
+  <xacro:insert_transmission name="yr_l_pel_joint"/>
+  <xacro:insert_transmission name="yr_l_hip_joint"/>
+  <xacro:insert_transmission name="yr_l_kne_joint"/>
+  <xacro:insert_transmission name="yr_l_ank_joint"/>
+  <xacro:insert_transmission name="yr_r_pel_joint"/>
+  <xacro:insert_transmission name="yr_r_hip_joint"/>
+  <xacro:insert_transmission name="yr_r_kne_joint"/>
+  <xacro:insert_transmission name="yr_r_ank_joint"/>
   <xacro:define_gazebo_material link_name="human_waist_link" r="0.7" g="0.7" b="0.7" a="1" mu="1.0" />
   <xacro:define_gazebo_material link_name="waist_link" r="0.7" g="0.7" b="0.7" a="1" mu="1.0"/>
@@ -187,15 +131,15 @@
   <xacro:define_gazebo_material link_name="l_thigh_link" r="0.7" g="0.7" b="0.7" a="1" mu="1.0"/>
   <xacro:define_gazebo_material link_name="l_shank_link" r="0.8" g="0.8" b="0.8" a="1" mu="1.0"/>
-  <xacro:define_gazebo_material link_name="l_foot_link" r="0.7" g="0.7" b="0.7" a="1" mu="3.0"/>
+  <xacro:define_gazebo_material link_name="l_foot_link" r="0.7" g="0.7" b="0.7" a="1" mu="1.0"/>
   <xacro:define_gazebo_material link_name="r_pel_link" r="0.7" g="0.7" b="0.7" a="1" mu="1.0"/>
   <xacro:define_gazebo_material link_name="r_thigh_link" r="0.7" g="0.7" b="0.7" a="1" mu="1.0"/>
   <xacro:define_gazebo_material link_name="r_shank_link" r="0.7" g="0.7" b="0.7" a="1" mu="1.0"/>
-  <xacro:define_gazebo_material link_name="r_foot_link" r="0.7" g="0.7" b="0.7" a="1" mu="3.0"/>
-<!--
+  <xacro:define_gazebo_material link_name="r_foot_link" r="0.7" g="0.7" b="0.7" a="1" mu="1.0"/>
+  <!--
   <xacro:define_gazebo_material link_name="stand_base" r="0.4" g="0.4" b="0.4" a="0.5" />
   <xacro:define_gazebo_material link_name="support_pole" r="0.4" g="0.4" b="0.4" a="0.5" />
  -->
   <!-- Use the macro to add IMU sensors to specific links -->
-  <!-- <xacro:add_imu_sensor link_name="l_pel_link" joint_name="yr_l_pel_joint" />
+  <xacro:add_imu_sensor link_name="l_pel_link" joint_name="yr_l_pel_joint" />
   <xacro:add_imu_sensor link_name="l_thigh_link" joint_name="yr_l_hip_joint" />
   <xacro:add_imu_sensor link_name="l_shank_link" joint_name="yr_l_kne_joint"/>
@@ -204,6 +148,6 @@
   <xacro:add_imu_sensor link_name="r_thigh_link" joint_name="yr_r_hip_joint"/>
   <xacro:add_imu_sensor link_name="r_shank_link" joint_name="yr_r_kne_joint"/>
-  <xacro:add_imu_sensor link_name="r_foot_link" joint_name="yr_r_ank_joint"/> -->
-<!--
+  <xacro:add_imu_sensor link_name="r_foot_link" joint_name="yr_r_ank_joint"/>
+  <!--
   <xacro:include filename="$(find realsense_ros_gazebo)/xacro/depthcam.xacro"/>
   <xacro:realsense_d435 sensor_name="d435_front" parent_link="l_thigh_link" rate="10">

File: src/yr_description/urdf/macros.xacro (robot description, xacro)
@@ -223,32 +223,24 @@
     </xacro:macro>
     <xacro:macro name="add_imu_sensor" params="link_name joint_name">
-        <gazebo reference="${link_name}">
-            <sensor type="imu" name="${link_name}_imu_sensor">
-                <pose>0 0 0 0 0 0</pose>
-                <always_on>true</always_on>
-                <update_rate>50</update_rate>
-                <imu>
-                    <angular_velocity>
-                        <x>0.0</x>
-                        <y>0.0</y>
-                        <z>0.0</z>
-                    </angular_velocity>
-                    <linear_acceleration>
-                        <x>0.0</x>
-                        <y>0.0</y>
-                        <z>0.0</z>
-                    </linear_acceleration>
-                </imu>
-                <plugin name="imu" filename="libgazebo_ros_imu_sensor.so">
-                    <ros>
-                        <!-- Output topic name -->
-                        <namespace>${joint_name}</namespace>
-                        <argument>imu/out:=imu</argument>
-                    </ros>
-                    <!-- Frame ID for the IMU data -->
-                    <frameName>${link_name}</frameName>
-                </plugin>
-            </sensor>
-        </gazebo>
+    <gazebo reference="${link_name}">
+        <gravity>true</gravity>
+        <sensor name="${joint_name}" type="imu">
+        <always_on>true</always_on>
+        <update_rate>100</update_rate>
+        <visualize>true</visualize>
+        <topic>${joint_name}/imu_data</topic>
+        <plugin filename="libgazebo_ros_imu_sensor.so" name="imu_plugin">
+            <topicName>${joint_name}/imu_data</topicName>
+            <bodyName>${joint_name}_imu</bodyName>
+            <updateRateHZ>10.0</updateRateHZ>
+            <gaussianNoise>0.0</gaussianNoise>
+            <xyzOffset>0 0 0</xyzOffset>
+            <rpyOffset>0 0 0</rpyOffset>
+            <frameName>${joint_name}_imu</frameName>
+            <initialOrientationAsReference>false</initialOrientationAsReference>
+        </plugin>
+        <pose>0 0 0 0 0 0</pose>
+        </sensor>
+    </gazebo>
     </xacro:macro>
 </robot>

File: src/yr_description/urdf/transmissions.xacro (robot description, xacro)
@@ -6,8 +6,8 @@
             <type>transmission_interface/SimpleTransmission</type>
             <joint name="${name}">
-                <hardwareInterface>hardware_interface/EffortJointInterface</hardwareInterface>
+                <hardwareInterface>EffortJointInterface</hardwareInterface>
             </joint>
             <actuator name="${name}_motor">
-                <hardwareInterface>EffortJointInterface</hardwareInterface>
+                <!-- <hardwareInterface>EffortJointInterface</hardwareInterface> -->
                 <mechanicalReduction>1</mechanicalReduction>
             </actuator>
