Commit message: Walking balance

File: src/yr_description/urdf/depth_cameras_setup.xacro (robot description, xacro)
@@ -24,5 +24,5 @@
 <joint name="d435_front_joint" type="fixed">
   <axis xyz="0 1 0" />
-  <origin xyz="${thigh_w/2} 0 ${-thigh_l/2}" rpy="0 0 0"/>
+  <origin xyz="${thigh_w/2} 0 ${-thigh_l/2}" rpy="0 ${0*PI/4} 0"/>
   <parent link="l_thigh_link"/>
   <child link="d435_front"/>

File: src/yr_description/urdf/exo.xacro (robot description, xacro)
@@ -8,10 +8,10 @@
 \
   <xacro:include filename="depth_cameras_setup.xacro" />
-  <!-- <link name="world"/>
+  <link name="world"/>
     <joint name="pole_to_waist" type="fixed">
         <parent link="world" />
         <child link="waist_link" />
-        <origin xyz="0 0 1.5" />
-    </joint> -->
+        <origin xyz="0 0 0" rpy="0 0 0"/>
+    </joint>
   <!--
   <link name="human_waist_link">
@@ -66,4 +66,31 @@
     </inertial>
   </link>
+  <link name="l_foot_bottom_link">
+    <!-- <collision>
+      <origin xyz="0 0 0" rpy="0 0 0" />
+      <geometry>
+        <box size="0.01 0.01 0.01" />
+      </geometry>
+      <origin xyz="0 0 0" rpy="0 0 0" />
+    </collision> -->
+    <visual>
+      <origin xyz="0 0 0" rpy="0 0 0" />
+      <geometry>
+        <box size="0.01 0.01 0.01" />
+      </geometry>
+      <origin xyz="0 0 0" rpy="0 0 0" />
+      <material name="${foot_mat}" />
+    </visual>
+    <inertial>
+      <origin xyz="0 0 0" rpy="0 0 0" />
+      <mass value="0.01" />
+      <inertia ixx="0.00001" ixy="0.0" ixz="0.0" iyy="0.00001" iyz="0.0" izz="0.00001" />
+    </inertial>
+  </link>
+  <joint name="l_foot_bottom_joint" type="fixed">
+    <parent link="l_foot_link" />
+    <child link="l_foot_bottom_link" />
+    <origin xyz="${foot_h/2} 0 ${-foot_h - foot_w/2}" rpy="0 0 0"/>
+  </joint>
   <xacro:create_link3 name="r_pel_link" m="${pel_m}" l="${pel_l}" w="${pel_w}" h="${pel_h}" o_x="${pel_x_offset}" o_y="${pel_y_offset}" o_z="${-pel_h_offset}" o_r="0" o_p="0" o_yaw="0" mat="${pel_mat}" mesh_filename="${pel_mesh}" mirror="1" />
   <xacro:create_link3 name="r_thigh_link" m="${thigh_m}" l="${thigh_l}" w="${thigh_w}" h="${thigh_h}" o_x="${-thigh_w}" o_y="${-thigh_w/2}" o_z="${-thigh_l}" o_r="0" o_p="0" o_yaw="0" mat="${thigh_mat}" mesh_filename="${thigh_mesh}" mirror="1" />
@@ -91,4 +118,31 @@
     </inertial>
   </link>
+  <link name="r_foot_bottom_link">
+    <!-- <collision>
+      <origin xyz="0 0 0" rpy="0 0 0" />
+      <geometry>
+        <box size="0.01 0.01 0.01" />
+      </geometry>
+      <origin xyz="0 0 0" rpy="0 0 0" />
+    </collision> -->
+    <visual>
+      <origin xyz="0 0 0" rpy="0 0 0" />
+      <geometry>
+        <box size="0.01 0.01 0.01" />
+      </geometry>
+      <origin xyz="0 0 0" rpy="0 0 0" />
+      <material name="${foot_mat}" />
+    </visual>
+    <inertial>
+      <origin xyz="0 0 0" rpy="0 0 0" />
+      <mass value="0.01" />
+      <inertia ixx="0.00001" ixy="0.0" ixz="0.0" iyy="0.00001" iyz="0.0" izz="0.00001" />
+    </inertial>
+  </link>
+  <joint name="r_foot_bottom_joint" type="fixed">
+    <parent link="r_foot_link" />
+    <child link="r_foot_bottom_link" />
+    <origin xyz="${foot_h/2} 0 ${-foot_h - foot_w/2}" rpy="0 0 0"/>
+  </joint>
   <!-- ======================================================= -->
   <!-- JOINTS                                                  -->
